File: KiCad/Base PCB.kicad_sch (KiCad schematic)
At the start: 8 parts, among them J201 Conn_02x32_Odd_Even, J202 Conn_02x20_Odd_Even

Commit message: Updated Schematic and PCB
Parts:
- renumbered GND201 to GND1, H201 to H1, H202 to H2, H203 to H3, H204 to H4, J201 to J3, J202 to J4, JP201 to JP3
Changed lines of the file:
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@@
   (symbol (lib_id "Mechanical:MountingHole_Pad") (at 50.8 165.1 0) (unit 1)
     (in_bom yes) (on_board yes)
-    (property "Reference" "H204" (id 0) (at 53.34 163.8554 0)
+    (property "Reference" "H4" (id 0) (at 53.34 163.8554 0)
       (effects (font (size 1.27 1.27)) (justify left))
     )
@@
   (symbol (lib_id "Mechanical:MountingHole_Pad") (at 31.75 165.1 0) (unit 1)
     (in_bom yes) (on_board yes)
-    (property "Reference" "GND201" (id 0) (at 34.29 163.8554 0)
+    (property "Reference" "GND1" (id 0) (at 34.29 163.8554 0)
       (effects (font (size 1.27 1.27)) (justify left))
     )
@@
   (symbol (lib_id "power:GND") (at 50.8 177.8 0) (unit 1)
     (in_bom yes) (on_board yes)
-    (property "Reference" "#PWR0201" (id 0) (at 50.8 184.15 0)
+    (property "Reference" "#PWR030" (id 0) (at 50.8 184.15 0)
       (effects (font (size 1.27 1.27)) hide)
     )
@@
   (symbol (lib_id "Device:Jumper_NO_Small") (at 50.8 172.72 270) (unit 1)
     (in_bom yes) (on_board yes)
-    (property "Reference" "JP201" (id 0) (at 52.0192 171.5516 90)
+    (property "Reference" "JP3" (id 0) (at 52.0192 171.5516 90)
       (effects (font (size 1.27 1.27)) (justify left))
     )
@@
   (symbol (lib_id "Mechanical:MountingHole") (at 50.8 158.75 0) (unit 1)
     (in_bom yes) (on_board yes)
-    (property "Reference" "H203" (id 0) (at 53.34 157.5816 0)
+    (property "Reference" "H3" (id 0) (at 53.34 157.5816 0)
       (effects (font (size 1.27 1.27)) (justify left))
     )
@@
   (symbol (lib_id "Mechanical:MountingHole") (at 50.8 153.67 0) (unit 1)
     (in_bom yes) (on_board yes)
-    (property "Reference" "H202" (id 0) (at 53.34 152.5016 0)
+    (property "Reference" "H2" (id 0) (at 53.34 152.5016 0)
       (effects (font (size 1.27 1.27)) (justify left))
     )
@@
   (symbol (lib_id "Mechanical:MountingHole") (at 50.8 148.59 0) (unit 1)
     (in_bom yes) (on_board yes)
-    (property "Reference" "H201" (id 0) (at 53.34 147.4216 0)
+    (property "Reference" "H1" (id 0) (at 53.34 147.4216 0)
       (effects (font (size 1.27 1.27)) (justify left))
     )
@@
   (symbol (lib_id "Connector_Generic:Conn_02x32_Odd_Even") (at 90.17 88.9 0) (mirror y) (unit 1)
     (in_bom yes) (on_board yes)
-    (property "Reference" "J201" (id 0) (at 88.9 45.2882 0))
+    (property "Reference" "J3" (id 0) (at 88.9 45.2882 0))
     (property "Value" "Conn_02x32_Odd_Even" (id 1) (at 88.9 47.5996 0))
     (property "Footprint" "Connector_PinSocket_2.54mm:PinSocket_2x32_P2.54mm_Vertical" (id 2) (at 90.17 88.9 0)
@@
   (symbol (lib_id "Connector_Generic:Conn_02x20_Odd_Even") (at 204.47 86.36 0) (mirror y) (unit 1)
     (in_bom yes) (on_board yes)
-    (property "Reference" "J202" (id 0) (at 203.2 57.9882 0))
+    (property "Reference" "J4" (id 0) (at 203.2 57.9882 0))
     (property "Value" "Conn_02x20_Odd_Even" (id 1) (at 203.2 60.2996 0))
     (property "Footprint" "Connector_PinSocket_2.54mm:PinSocket_2x20_P2.54mm_Vertical" (id 2) (at 204.47 86.36 0)

Commit message: Update Schematic and PCB
Parts:
- renumbered JP3 to JP2
Changed lines of the file:
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@@
   (symbol (lib_id "power:GND") (at 50.8 177.8 0) (unit 1)
     (in_bom yes) (on_board yes)
-    (property "Reference" "#PWR036" (id 0) (at 50.8 184.15 0)
+    (property "Reference" "#PWR035" (id 0) (at 50.8 184.15 0)
       (effects (font (size 1.27 1.27)) hide)
     )
@@
   (symbol (lib_id "Device:Jumper_NO_Small") (at 50.8 172.72 270) (unit 1)
     (in_bom yes) (on_board yes)
-    (property "Reference" "JP3" (id 0) (at 52.0192 171.5516 90)
+    (property "Reference" "JP2" (id 0) (at 52.0192 171.5516 90)
       (effects (font (size 1.27 1.27)) (justify left))
     )
